Commit message: Symbol name update

File: pybullet/robotiq-3f-gripper_articulated.urdf (robot description, URDF)
Before this commit: robot robotiq-3f-gripper_articulated, 13 links, 12 joints
Links:
- removed link finger_1_link_0
- removed link finger_1_link_1
- removed link finger_1_link_2
- removed link finger_1_link_3
- removed link finger_2_link_0
- removed link finger_2_link_1
- removed link finger_2_link_2
- removed link finger_2_link_3
- removed link finger_middle_link_0
- removed link finger_middle_link_1
- removed link finger_middle_link_2
- removed link finger_middle_link_3
- added link finger_A_link_0, mass 0.05; collision mesh filename=meshes/robotiq-3f-gripper_articulated/collision/link_0.STL; visual mesh filename=meshes/robotiq-3f-gripper_articulated/visual/link_0.dae
- added link finger_A_link_1, mass 0.15; collision mesh filename=meshes/robotiq-3f-gripper_articulated/collision/link_1.STL; visual mesh filename=meshes/robotiq-3f-gripper_articulated/visual/link_1.dae
- added link finger_A_link_2, mass 0.15; collision mesh filename=meshes/robotiq-3f-gripper_articulated/collision/link_2.STL; visual mesh filename=meshes/robotiq-3f-gripper_articulated/visual/link_2.dae
- added link finger_A_link_3, mass 0.05; collision mesh filename=meshes/robotiq-3f-gripper_articulated/collision/link_3.STL; visual mesh filename=meshes/robotiq-3f-gripper_articulated/visual/link_3.dae
- added link finger_B_link_0, mass 0.05; collision mesh filename=meshes/robotiq-3f-gripper_articulated/collision/link_0.STL; visual mesh filename=meshes/robotiq-3f-gripper_articulated/visual/link_0.dae
- added link finger_B_link_1, mass 0.15; collision mesh filename=meshes/robotiq-3f-gripper_articulated/collision/link_1.STL; visual mesh filename=meshes/robotiq-3f-gripper_articulated/visual/link_1.dae
- added link finger_B_link_2, mass 0.15; collision mesh filename=meshes/robotiq-3f-gripper_articulated/collision/link_2.STL; visual mesh filename=meshes/robotiq-3f-gripper_articulated/visual/link_2.dae
- added link finger_B_link_3, mass 0.05; collision mesh filename=meshes/robotiq-3f-gripper_articulated/collision/link_3.STL; visual mesh filename=meshes/robotiq-3f-gripper_articulated/visual/link_3.dae
- added link finger_C_link_0, mass 0.05; collision mesh filename=meshes/robotiq-3f-gripper_articulated/collision/link_0.STL; visual mesh filename=meshes/robotiq-3f-gripper_articulated/visual/link_0.dae
- added link finger_C_link_1, mass 0.15; collision mesh filename=meshes/robotiq-3f-gripper_articulated/collision/link_1.STL; visual mesh filename=meshes/robotiq-3f-gripper_articulated/visual/link_1.dae
- added link finger_C_link_2, mass 0.15; collision mesh filename=meshes/robotiq-3f-gripper_articulated/collision/link_2.STL; visual mesh filename=meshes/robotiq-3f-gripper_articulated/visual/link_2.dae
- added link finger_C_link_3, mass 0.05; collision mesh filename=meshes/robotiq-3f-gripper_articulated/collision/link_3.STL; visual mesh filename=meshes/robotiq-3f-gripper_articulated/visual/link_3.dae
Joints:
- removed joint finger_1_joint_1
- removed joint finger_1_joint_2
- removed joint finger_1_joint_3
- removed joint finger_2_joint_1
- removed joint finger_2_joint_2
- removed joint finger_2_joint_3
- removed joint finger_middle_joint_1
- removed joint finger_middle_joint_2
- removed joint finger_middle_joint_3
- removed joint palm_finger_1_joint
- removed joint palm_finger_2_joint
- removed joint palm_finger_middle_joint
- added joint finger_A_joint_1: type revolute, parent finger_A_link_0, child finger_A_link_1, origin xyz=0.020 0 0 rpy=0 0 0, axis 0 0 1, limit lower=0 upper=1.2217 effort=100 velocity=100
- added joint finger_A_joint_2: type revolute, parent finger_A_link_1, child finger_A_link_2, origin xyz=0.050 -.028 0 rpy=0 0 -0.47124, axis 0 0 1, limit lower=0 upper=1.5708 effort=100 velocity=100
- added joint finger_A_joint_3: type revolute, parent finger_A_link_2, child finger_A_link_3, origin xyz=0.039 0 0 rpy=0 0 0, axis 0 0 1, limit lower=-0.90757 upper=0.80285 effort=100 velocity=100
- added joint finger_B_joint_1: type revolute, parent finger_B_link_0, child finger_B_link_1, origin xyz=0.020 0 0 rpy=0 0 0, axis 0 0 1, limit lower=0 upper=1.2217 effort=100 velocity=100
- added joint finger_B_joint_2: type revolute, parent finger_B_link_1, child finger_B_link_2, origin xyz=0.050 -.028 0 rpy=0 0 -0.47124, axis 0 0 1, limit lower=0 upper=1.5708 effort=100 velocity=100
- added joint finger_B_joint_3: type revolute, parent finger_B_link_2, child finger_B_link_3, origin xyz=0.039 0 0 rpy=0 0 0, axis 0 0 1, limit lower=-0.90757 upper=0.80285 effort=100 velocity=100
- added joint finger_C_joint_1: type revolute, parent finger_C_link_0, child finger_C_link_1, origin xyz=0.020 0 0 rpy=0 0 0, axis 0 0 1, limit lower=0 upper=1.2217 effort=100 velocity=100
- added joint finger_C_joint_2: type revolute, parent finger_C_link_1, child finger_C_link_2, origin xyz=0.050 -.028 0 rpy=0 0 -0.47124, axis 0 0 1, limit lower=0 upper=1.5708 effort=100 velocity=100
- added joint finger_C_joint_3: type revolute, parent finger_C_link_2, child finger_C_link_3, origin xyz=0.039 0 0 rpy=0 0 0, axis 0 0 1, limit lower=-0.90757 upper=0.80285 effort=100 velocity=100
- added joint palm_finger_A_joint: type fixed, parent palm, child finger_A_link_0, origin xyz=0.0455 0.0214 0 rpy=0 0 1.5708, axis 0 0 1
- added joint palm_finger_B_joint: type revolute, parent palm, child finger_B_link_0, origin xyz=-0.0455 0.0214 -0.036 rpy=0 3.1416 -1.5708, axis 0 1 0, limit lower=-0.27925 upper=0.17453 effort=100 velocity=100
- added joint palm_finger_C_joint: type revolute, parent palm, child finger_C_link_0, origin xyz=-0.0455 0.0214 0.036 rpy=0 3.1416 -1.5708, axis 0 1 0, limit lower=-0.17453 upper=0.27925 effort=100 velocity=100
